Commit message: add sim objects, start

File: src/condynsate/__assets__/gyro.urdf (robot description, URDF)
Before this commit: robot gyro, 5 links, 4 joints
Joints:
- joint base_to_outer: origin xyz=0 0 1.6 rpy=0 0 0 -> xyz=0 0 -1.6 rpy=0 1.5708 0
- joint outer_to_r2: origin xyz=0 0 0 rpy=0 0 0 -> xyz=0 0 0 rpy=0 1.5708 0

Commit message: started project.py

File: src/condynsate/__assets__/gyro.urdf (robot description, URDF)
Before this commit: robot gyro, 5 links, 4 joints
Joints:
- joint base_to_outer: origin xyz=0 0 -1.6 rpy=0 1.5708 0 -> xyz=0 0 1.6 rpy=0 -1.5708 1.5708
