Commit message: added await keypress

File: src/condynsate/__assets__/plane_big.urdf (robot description, URDF)
Before this commit: robot plane, 1 links, 0 joints
Links:
- link plane: geometry collision box size=100 100 1; visual mesh filename=plane.obj scale=100 100 1

File: src/condynsate/__assets__/plane_medium.urdf (robot description, URDF)
Before this commit: robot plane_medium, 1 links, 0 joints
Links:
- link plane: geometry collision box size=10 10 1; visual mesh filename=plane.obj scale=10 10 1

File: src/condynsate/__assets__/plane_small.urdf (robot description, URDF)
Before this commit: robot plane_small, 1 links, 0 joints
Links:
- link plane: geometry collision box size=1 1 1; visual mesh filename=plane.obj scale=1 1 1
