Commit message: added wheel project

File: src/condynsate/__assets__/wheel.urdf (robot description, URDF)
Before this commit: robot wheel, 5 links, 4 joints
Links:
- link wheel: geometry visual mesh filename=hubbed_wheel_1x0.1_lower_origin.stl scale=0.5 0.5 0.5
Joints:
- joint axle_to_target: axis 0 0 1 -> 0 1 0
