Commit message: gyro example, joint axis bug

File: src/condynsate/__assets__/cart.urdf (robot description, URDF)
Before this commit: robot cart, 7 links, 6 joints
Links:
- link arm: geometry collision mesh filename=Cylinder_1x1_lower_origin.stl scale=0.05 0.05 1; visual mesh filename=Cylinder_1x1_lower_origin.stl scale=0.05 0.05 1
- link chassis: mass 2.0 -> 2; geometry collision mesh filename=Cube_1x1x1_lower_origin.stl scale=1 0.5 0.25; visual mesh filename=Cube_1x1x1_lower_origin.stl scale=1 0.5 0.25
- link mass: mass 1.0 -> 1; geometry collision mesh filename=Sphere_1_center_origin.stl scale=0.2 0.2 0.2; visual mesh filename=Sphere_1_center_origin.stl scale=0.2 0.2 0.2
- link wheel_1: geometry collision mesh filename=Cylinder_1x1_lower_origin.stl scale=0.25 0.25 0.05; visual mesh filename=Cylinder_1x1_lower_origin.stl scale=0.25 0.25 0.05
- link wheel_2: geometry collision mesh filename=Cylinder_1x1_lower_origin.stl scale=0.25 0.25 0.05; visual mesh filename=Cylinder_1x1_lower_origin.stl scale=0.25 0.25 0.05
- link wheel_3: geometry collision mesh filename=Cylinder_1x1_lower_origin.stl scale=0.25 0.25 0.05; visual mesh filename=Cylinder_1x1_lower_origin.stl scale=0.25 0.25 0.05
- link wheel_4: geometry collision mesh filename=Cylinder_1x1_lower_origin.stl scale=0.25 0.25 0.05; visual mesh filename=Cylinder_1x1_lower_origin.stl scale=0.25 0.25 0.05
Joints:
- joint arm_to_mass: origin xyz=0 0 1.0 rpy=0 0 0 -> xyz=0 0 1 rpy=0 0 0
- joint chassis_to_arm: origin xyz=0 0 0.125 rpy=0 0 0 -> xyz=0 0 0.25 rpy=0 0 0
- joint chassis_to_wheel_1: axis 0 0 1 -> 0 0 -1; origin xyz=0.375 -0.275 -0.125 rpy=1.5707963267948966 0 0 -> xyz=-0.375 -0.251 0 rpy=1.5708 0 0
- joint chassis_to_wheel_2: axis 0 0 1 -> 0 0 -1; origin xyz=-0.375 -0.275 -0.125 rpy=1.5707963267948966 0 0 -> xyz=0.375 -0.251 0 rpy=1.5708 0 0
- joint chassis_to_wheel_3: origin xyz=-0.375 0.275 -0.125 rpy=1.5707963267948966 0 0 -> xyz=-0.375 0.251 0 rpy=-1.5708 0 0
- joint chassis_to_wheel_4: origin xyz=0.375 0.275 -0.125 rpy=1.5707963267948966 0 0 -> xyz=0.375 0.251 0 rpy=-1.5708 0 0

File: src/condynsate/__assets__/cube.urdf (robot description, URDF)
Before this commit: robot cube, 1 links, 0 joints
Links:
- link cube: mass 1.0 -> 1; geometry collision mesh filename=Cube_1x1x1_center_origin.stl scale=1 1 1; visual mesh filename=Cube_1x1x1_center_origin.stl scale=1 1 1

File: src/condynsate/__assets__/double_pendulum.urdf (robot description, URDF)
Before this commit: robot pendulum, 5 links, 4 joints
Links:
- removed link arm1
- removed link arm2
- removed link chassis
- removed link mass1
- removed link mass2
- added link arm_1, mass 0; visual mesh filename=Cylinder_1x1_lower_origin.stl scale=0.05 0.05 1.0
- added link arm_2, mass 0; visual mesh filename=Cylinder_1x1_lower_origin.stl scale=0.05 0.05 1.0
- added link base, mass 0; visual mesh filename=Cube_1x1x1_lower_origin.stl scale=0.1 0.1 0.1
- added link mass_1, mass 1; visual mesh filename=Sphere_1_center_origin.stl scale=0.2 0.2 0.2
- added link mass_2, mass 1; visual mesh filename=Sphere_1_center_origin.stl scale=0.2 0.2 0.2
Joints:
- removed joint arm1_to_mass1
- removed joint arm2_to_mass2
- removed joint chassis_to_arm1
- removed joint mass1_to_arm2
- added joint arm_1_to_mass_1: type fixed, parent arm_1, child mass_1, origin xyz=0 0 1 rpy=0 0 0
- added joint arm_2_to_mass_2: type fixed, parent arm_2, child mass_2, origin xyz=0 0 1 rpy=0 0 0
- added joint base_to_arm_1: type continuous, parent base, child arm_1, origin xyz=0 0 0 rpy=0 0 0, axis 0 -1 0
- added joint mass_1_to_arm_2: type continuous, parent mass_1, child arm_2, origin xyz=0 0 0 rpy=0 0 0, axis 0 -1 0

File: src/condynsate/__assets__/gyro.urdf (robot description, URDF)
Before this commit: robot gyro, 5 links, 4 joints
Links:
- removed link outer
- removed link r1
- removed link r2
- added link ring1, mass 0.16; visual mesh filename=gyroring_0.6-ODx0.3-ID_center_origin.stl scale=2 2 2
- added link ring2, mass 0.16; visual mesh filename=gyroring_0.9-ODx0.6-ID_center_origin.stl scale=2 2 2
- added link ring3, mass 0.16; visual mesh filename=gyroouter_1-ODx0.9ID_lower_origin.stl scale=2 2 2
- link base: geometry visual mesh filename=Cylinder_1x1_lower_origin.stl scale=1 1 0.1
- link core: mass 1.0 -> 8; geometry visual mesh filename=gyrocore.stl scale=2 2 2
Joints:
- removed joint base_to_outer
- removed joint outer_to_r2
- removed joint r1_to_core
- removed joint r2_to_r1
- added joint base_to_ring3: type continuous, parent base, child ring3, origin xyz=0 0 0.1 rpy=0 0 0, axis 0 0 1
- added joint ring1_to_core: type continuous, parent ring1, child core, origin xyz=0 0 0 rpy=0 0 0, axis 0 0 1
- added joint ring2_to_ring1: type continuous, parent ring2, child ring1, origin xyz=0 0 0 rpy=0 0 0, axis 0 1 0
- added joint ring3_to_ring2: type continuous, parent ring3, child ring2, origin xyz=0 0 2 rpy=0 0 0, axis 1 0 0

File: src/condynsate/__assets__/pendulum.urdf (robot description, URDF)
Before this commit: robot pendulum, 3 links, 2 joints
Links:
- removed link chassis
- added link base, mass 0; visual mesh filename=Cube_1x1x1_lower_origin.stl scale=0.1 0.1 0.1
- link arm: mass 0.0 -> 0; geometry visual mesh filename=Cylinder_1x1_lower_origin.stl scale=0.05 0.05 1.0
- link mass: mass 1.0 -> 1; geometry visual mesh filename=Sphere_1_center_origin.stl scale=0.2 0.2 0.2
Joints:
- removed joint chassis_to_arm
- added joint base_to_arm: type continuous, parent base, child arm, origin xyz=0 0 0 rpy=0 0 0, axis 0 -1 0

Commit message: added pendulum cart proj 1

File: src/condynsate/__assets__/cart.urdf (robot description, URDF)
Before this commit: robot cart, 7 links, 6 joints
Links:
- link chassis: mass 2 -> 23.5
- link mass: mass 1 -> 4.0
- link wheel_1: mass 0.25 -> 1.8
- link wheel_2: mass 0.25 -> 1.8
- link wheel_3: mass 0.25 -> 1.8
- link wheel_4: mass 0.25 -> 1.8
