Commit message: gryo proj edits

File: src/condynsate/__assets__/dual_axis_cmg.urdf (robot description, URDF)
Before this commit: robot gyro, 5 links, 4 joints
Links:
- removed link base
- removed link ring1
- removed link ring2
- removed link ring3
- added link chassis, mass 3.06; visual mesh filename=spacecraft_chassis_1OD_0.9ID.stl scale=2 2 2
- added link inner_gimbal, mass 0.119; visual mesh filename=gyroring_0.6-ODx0.3-ID_center_origin.stl scale=2 2 2
- added link outer_gimbal, mass 0.221; visual mesh filename=gyroring_0.9-ODx0.6-ID_center_origin.stl scale=2 2 2
- link core: mass 8 -> 0.343
Joints:
- removed joint base_to_ring3
- removed joint ring1_to_core
- removed joint ring2_to_ring1
- removed joint ring3_to_ring2
- added joint chassis_to_outer: type continuous, parent chassis, child outer_gimbal, origin xyz=0 0 0 rpy=0 0 0, axis 1 0 0
- added joint inner_to_core: type continuous, parent inner_gimbal, child core, origin xyz=0 0 0 rpy=0 0 0, axis 1 0 0
- added joint outer_to_inner: type continuous, parent outer_gimbal, child inner_gimbal, origin xyz=0 0 0 rpy=0 0 0, axis 0 1 0
