Commit message: proj updates, added self collision arg

File: src/condynsate/__assets__/single_axis_cmg.urdf (robot description, URDF)
Before this commit: robot gyro, 6 links, 5 joints
Links:
- removed link baserod
- removed link chassis
- removed link core
- removed link inner_gimbal
- removed link outer_gimbal
- added link A, mass 0.221; visual mesh filename=gyroring_18-Wx14-ODx12-IDx2-T_cen_orig.stl scale=0.1 0.1 0.1
- added link B, mass 0.119; visual mesh filename=gyroring_12-Wx8-ODx6-IDx2-T_cen-orig.stl scale=0.1 0.1 0.1
- added link flywheel, mass 0.622; visual mesh filename=gyrocore_6-Wx5.5-ODx3-T_cen-orig.stl scale=0.1 0.1 0.1
- added link mass, mass 0.0221; visual mesh filename=Sphere_1_center_origin.stl scale=0.25 0.25 0.25
- added link massrod, mass 0; collision mesh filename=Cylinder_1x1_lower_origin.stl scale=0.1 0.1 0.7; visual mesh filename=Cylinder_1x1_lower_origin.stl scale=0.1 0.1 0.7
- link base: geometry collision mesh filename=gyrochassis-fixed_20-ODx18ID_cen_orig.stl scale=0.1 0.1 0.1; visual mesh filename=gyrochassis-fixed_20-ODx18ID_cen_orig.stl scale=0.1 0.1 0.1
Joints:
- removed joint base_to_baserod
- removed joint baserod_to_chassis
- removed joint chassis_to_outer
- removed joint inner_to_core
- removed joint outer_to_inner
- added joint A_to_B: type continuous, parent A, child B, origin xyz=0 0 0 rpy=0 0 0, axis 0 0 1
- added joint A_to_massrod: type fixed, parent A, child massrod, origin xyz=0 0 0.7 rpy=0 0 0
- added joint B_to_flywheel: type continuous, parent B, child flywheel, origin xyz=0 0 0 rpy=0 0 0, axis 1 0 0
- added joint base_to_A: type continuous, parent base, child A, origin xyz=0 0 0 rpy=0 0 0, axis 0 1 0
- added joint massrod_to_mass: type fixed, parent massrod, child mass, origin xyz=0 0 0.8 rpy=0 0 0
