Commit message: cmg proj wip

File: src/condynsate/__assets__/parallel_single_axis_cmg.urdf (robot description, URDF)
Before this commit: robot gyro, 5 links, 4 joints
Links:
- link Fa: mass 0.770 -> 2.49
- link Fb: mass 0.770 -> 2.49
Joints:
- joint S_to_A: origin xyz=-0.95 0 0 rpy=0 0 0 -> xyz=-0.95 0 0 rpy=0 0 1.5708
- joint S_to_B: origin xyz=0.95 0 0 rpy=0 0 0 -> xyz=0.95 0 0 rpy=0 0 1.5708

Commit message: added emissivity to visualizer

File: src/condynsate/__assets__/parallel_single_axis_cmg.urdf (robot description, URDF)
Before this commit: robot gyro, 5 links, 4 joints
Links:
- link A: geometry visual mesh filename=gyroring_XZ-Y_18-Wx14-ODx12-IDx2-T_cen_orig.stl scale=0.1 0.1 0.1
- link B: geometry visual mesh filename=gyroring_XZ-Y_18-Wx14-ODx12-IDx2-T_cen_orig.stl scale=0.1 0.1 0.1
- link Fa: mass 2.49 -> 3.63; geometry visual mesh filename=gyrocore_XZ-Y_6-Wx11.5-ODx4-T_cen-orig.stl scale=0.1 0.1 0.1
- link Fb: mass 2.49 -> 3.63; geometry visual mesh filename=gyrocore_XZ-Y_6-Wx11.5-ODx4-T_cen-orig.stl scale=0.1 0.1 0.1
Joints:
- joint A_to_Fa: axis 1 0 0 -> 0 1 0
- joint B_to_Fb: axis 1 0 0 -> 0 1 0
- joint S_to_A: origin xyz=-0.95 0 0 rpy=0 0 1.5708 -> xyz=-0.95 0 0 rpy=0 0 0
- joint S_to_B: origin xyz=0.95 0 0 rpy=0 0 1.5708 -> xyz=0.95 0 0 rpy=0 0 0

Commit message: visual edits to par cmg proj

File: src/condynsate/__assets__/parallel_single_axis_cmg.urdf (robot description, URDF)
Before this commit: robot gyro, 5 links, 4 joints
Links:
- link S: geometry visual mesh filename=dual_CMG_spacecraft_19-ODx18-ID_cen-orig.obj scale=0.1 0.1 0.1
