Commit message: format gyro .stl names

File: src/condynsate/__assets__/gyroscope.urdf (robot description, URDF)
Before this commit: robot gyro, 5 links, 4 joints
Links:
- removed link chassis
- removed link core
- removed link inner_gimbal
- removed link outer_gimbal
- added link A, mass 0.322; visual mesh filename=gyrochassis-rotational_XZ-Z_20-Hx20-ODx18-IDx2-T_cen-orig.s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 scale=0.1 0.1 0.1
- added link B, mass 0.221; visual mesh filename=gyroring_XY-X_18-Wx14-ODx12-IDx2-T_cen-orig.stl scale=0.1 0.1 0.1
- added link C, mass 0.119; visual mesh filename=gyroring_YZ-Y_12-Wx8-ODx6-IDx2-T_cen-orig.stl scale=0.1 0.1 0.1
- added link flywheel, mass 0.622; visual mesh filename=gyrocore_XY-Z_6-Wx5.5-ODx3-T_cen-orig.stl scale=0.1 0.1 0.1
Joints:
- removed joint base_to_chassis
- removed joint chassis_to_outer
- removed joint inner_to_core
- removed joint outer_to_inner
- added joint A_to_B: type continuous, parent A, child B, origin xyz=0 0 0 rpy=0 0 0, axis 1 0 0
- added joint B_to_C: type continuous, parent B, child C, origin xyz=0 0 0 rpy=0 0 0, axis 0 1 0
- added joint C_to_flywheel: type continuous, parent C, child flywheel, origin xyz=0 0 0 rpy=0 0 0, axis 0 0 1
- added joint base_to_A: type continuous, parent base, child A, origin xyz=0 0 2 rpy=0 0 0, axis 0 0 1

File: src/condynsate/__assets__/opposed_sacmg.urdf (robot description, URDF)
Before this commit: robot parallel_sacmg_spacecraft, 5 links, 4 joints
Links:
- link A: geometry visual mesh filename=gyroring_XZ-Y_18-Wx14-ODx12-IDx2-T_cen-orig.stl scale=0.1 0.1 0.1
- link B: geometry visual mesh filename=gyroring_XZ-Y_18-Wx14-ODx12-IDx2-T_cen-orig.stl scale=0.1 0.1 0.1
- link S: geometry visual mesh filename=opposed-gyrochassis-spacecraft_19-ODx18-ID_cen-orig.obj scale=0.1 0.1 0.1

File: src/condynsate/__assets__/sacmg.urdf (robot description, URDF)
Before this commit: robot gyro, 6 links, 5 joints
Links:
- link A: geometry visual mesh filename=gyroring_YZ-Y_18-Wx14-ODx12-IDx2-T_cen-orig.stl scale=0.1 0.1 0.1
- link B: geometry visual mesh filename=gyroring_XZ-Z_12-Wx8-ODx6-IDx2-T_cen-orig.stl scale=0.1 0.1 0.1
- link base: geometry visual mesh filename=gyrochassis-fixed_20-ODx18-ID_cen-orig.stl scale=0.1 0.1 0.1
- link flywheel: geometry visual mesh filename=gyrocore_YZ-X_6-Wx5.5-ODx3-T_cen-orig.stl scale=0.1 0.1 0.1
