Commit message: update link set_color+texture

File: src/condynsate/__assets__/sphere.urdf (robot description, URDF)
Before this commit: robot cube, 1 links, 0 joints
Links:
- removed link cube
- added link sphere, mass 1; collision mesh filename=Sphere_1_center_origin.stl scale=1 1 1; visual mesh filename=Sphere_1_center_origin.stl scale=1 1 1
