Commit message: stitched textures now added

File: src/condynsate/__assets__/cessna172.urdf (robot description, URDF)
Before this commit: robot cessna172, 10 links, 9 joints
Links:
- link elevator: geometry visual mesh filename=airplane_elevator.obj scale=1 1 1
- link flaps: geometry visual mesh filename=airplane_flaps.obj scale=1 1 1
- link fuselage: mass 964. -> 964.0; geometry visual mesh filename=airplane_fuselage.obj scale=1 1 1
- link l_aileron: geometry visual mesh filename=airplane_l_aileron.obj scale=1 1 1
- link nosecone: geometry visual mesh filename=airplane_nosecone.obj scale=1 1 1
- link prop: geometry visual mesh filename=airplane_prop.obj scale=1 1 1
- link r_aileron: geometry visual mesh filename=airplane_r_aileron.obj scale=1 1 1
- link rudder: geometry visual mesh filename=airplane_rudder.obj scale=1 1 1
- link wheels: geometry visual mesh filename=airplane_wheels.obj scale=1 1 1
- link windows: geometry visual mesh filename=airplane_windows.obj scale=1 1 1
Joints:
- joint fuselage_to_elevator: origin xyz=-0.5029 0 -0.0045047 rpy=0 0 0 -> xyz=-5.029 0 -0.045047 rpy=0 0 0
- joint fuselage_to_flaps: origin xyz=-0.10464 0 0.070631 rpy=0 0 0 -> xyz=-1.0464 0 0.70631 rpy=0 0 0
- joint fuselage_to_l_aileron: origin xyz=-0.091651 0.40841 0.087295 rpy=0 0 0 -> xyz=-0.91651 4.0841 0.87295 rpy=0 0 0
- joint fuselage_to_nosecone: origin xyz=0.20309 0 0.0271 rpy=0 0 0 -> xyz=2.0309 0 0.271 rpy=0 0 0
- joint fuselage_to_r_aileron: origin xyz=-0.091651 -0.40841 0.087295 rpy=0 0 0 -> xyz=-0.91651 -4.0841 0.87295 rpy=0 0 0
- joint fuselage_to_rudder: origin xyz=-0.54586 0.001 0.0656 rpy=0 0 0 -> xyz=-5.4586 0.01 0.656 rpy=0 0 0

Commit message: fix chase cam, add stall buffet

File: src/condynsate/__assets__/cessna172.urdf (robot description, URDF)
Before this commit: robot cessna172, 10 links, 9 joints
Links:
- link fuselage: mass 964.0 -> 950.0
- link prop: mass 0 -> 14.0

Commit message: viz perf imp

File: src/condynsate/__assets__/cessna172.urdf (robot description, URDF)
Before this commit: robot cessna172, 10 links, 9 joints
Joints:
- joint fuselage_to_nosecone: origin xyz=2.0309 0 0.271 rpy=0 0 0 -> xyz=2.0834, 0, 0.26758 rpy=0 0 0

Commit message: fix CoM to W tnsfrm

File: src/condynsate/__assets__/cessna172.urdf (robot description, URDF)
Before this commit: robot cessna172, 10 links, 9 joints
Links:
- link fuselage: mass 950.0 -> 964.0
- link prop: mass 14.0 -> 0

Commit message: added collision to cessna 172

File: src/condynsate/__assets__/cessna172.urdf (robot description, URDF)
Before this commit: robot cessna172, 10 links, 9 joints
Links:
- link elevator: geometry collision mesh filename=airplane_elevator.obj scale=1 1 1; visual mesh filename=airplane_elevator.obj scale=1 1 1
- link fuselage: geometry collision mesh filename=airplane_fuselage.obj scale=1 1 1; visual mesh filename=airplane_fuselage.obj scale=1 1 1
- link rudder: geometry collision mesh filename=airplane_rudder.obj scale=1 1 1; visual mesh filename=airplane_rudder.obj scale=1 1 1
- link wheels: geometry collision mesh filename=airplane_wheels.obj scale=1 1 1; visual mesh filename=airplane_wheels.obj scale=1 1 1
